File: Wiring & PCB/Wiring/Wiring.sch (KiCad schematic (older format))
At the start: 1 part

Commit message: updates to the wiring design
Parts:
- added 470ohm (x3): R_US, symbol Device:R_US
- added D0, D1, D2: LED, symbol Device:LED
- added LS001: warnPiezo, symbol Device:Speaker_Crystal
- added M0, M1: Motor_DC, symbol Motor:Motor_DC
- added M2: Stepper_Motor_unipolar_6pin, symbol Motor:Stepper_Motor_unipolar_6pin
- added RV?: R_POT, symbol Device:R_POT
- added SW0: Ascention Limit 1, symbol Switch:SW_DPST_x2
- added SW1: Ascention Limit 2, symbol Switch:SW_DPST_x2
- added SW2: Declination Limit 1, symbol Switch:SW_DPST_x2
- added SW?: Resolution Switch, symbol Switch:SW_DPST_x2
- added SW?: Function Switch, symbol Switch:SW_SPDT_MSM
- added U (x2): AMT-22, symbol Device:AMT-22
- added U1: Ardunio_Micro, symbol Device:Ardunio_Micro
- added U3: ULN2004A, symbol Transistor_Array:ULN2004A
- added U4: pchero_dualH, symbol Device:pchero_dualH
- added U?: 20x4_Adafriuit_lcd, symbol Device:20x4_Adafriuit_lcd
- gave numbers to parts that had none: 1
Connections:
- net motorBpwm: now reaches U0.10 (D10)
- net motorBpwm: now also U4.~ (OUT4)
- net at U0.11 (D11): now also U4.~ (OUT4)
- net at U0.12 (D12): now also U4.~ (OUT4)
- net motorApwm: now reaches U0.13 (D13)
- net motorApwm: now also U4.~ (OUT4)
- net at U0.15 (RX3): now also SW2.2 (B)
- net at U0.16 (TX2): now also SW1.2 (B)
- net at U0.17 (RX2): now also SW0.2 (B)
- net at U0.18 (TX1): now also U1.~ (~RESET)
- net at U0.19 (RX1): now also U1.~ (~RESET)
- net at U0.2 (D2): now also U.6 (MCLR)
- net heater_LED: now reaches U0.26 (D26)
- net heater_LED: now also D0.2 (A)
- net track_LED: now reaches U0.27 (D27)
- net track_LED: now also D1.2 (A)
- net 47_to_warn: now reaches U0.28 (D28)
- net 47_to_warn: now also LS001.1
- net estop_LED: now reaches U0.29 (D29)
- net estop_LED: now also D2.2 (A)
- net at U0.3 (D3): now also U.6 (MCLR)
- net at U0.50 (D50): now also U.5 (MODE), U.5 (MODE)
- net at U0.51 (D51): now also U.3 (A), U.3 (A)
- net at U0.52 (D52): now also U.2 (B), U.2 (B)
- net at U0.8 (D8): now also U4.~ (OUT4)
- net at U0.9 (D9): now also U4.~ (OUT4)
- net Earth: now reaches U0.~ (VIN)
- net Earth: now also 470ohm.1, 470ohm.1, 470ohm.1, LS001.2, U.4 (GND), U.4 (GND), U4.~ (OUT4)
- new net: U.1 (+5v), U.1 (+5v), U0.~ (VIN), U4.~ (OUT4)
- new net: SW0.1 (A), SW1.1 (A), SW2.1 (A), U0.~ (VIN)
- new net: M0.1 (+), U4.~ (OUT4)
- new net: M0.2 (-), U4.~ (OUT4)
- new net: M1.1 (+), U4.~ (OUT4)
- new net: M1.2 (-), U4.~ (OUT4)
- new net: 470ohm.2, D0.1 (K)
- new net: 470ohm.2, D1.1 (K)
- new net: 470ohm.2, D2.1 (K)
- new net: U1.13 (D13), U?.4 (RS)
- new net: U1.A10 (D10/PB6), U?.13 (DB6)
- new net: U1.A11 (D12/PD6), U?.6 (E)
- new net: SW?.3, U1.A7 (D6/PD7/PWM)
- new net: U1.A8 (D8/PB4), U?.11 (DB4)
- new net: U1.A9 (D9/PB5), U?.12 (DB5)
- new net: RV?.3, U1.~ (~RESET), U?.1 (VSS), U?.16 (LED-), U?.5 (R/W)
- new net: U1.~ (~RESET), U?.14 (DB7)
- new net: RV?.1, SW?.1 (A), SW?.2, U1.~ (~RESET), U?.15 (LED+), U?.2 (VDD)
- new net: SW?.2 (B), U1.~ (~RESET)
- new net: SW?.1, U1.~ (~RESET)
- new net: RV?.2, U?.3 (V0)
- new net: M2.1, U3.15 (O2)
- new net: M2.2, M2.5, U3.9 (COM)
- new net: M2.3 (-), U3.16 (O1)
- new net: M2.4, U3.4 (I4)
- new net: M2.6, U3.3 (I3)
- new net +9V: U4.~ (OUT4)
Other:
- note added: "+- 5v supplied via usb\n"
- note added: "CONTRAST POT\n"
- note added: "Fix this so multiple switches can be down at once\n"
- note added: "Separate power system.\nMotors take 0-9.5V"
- moved on the sheet: U0

Commit message: wiring updates
Parts:
- added U?: Joystick, symbol Device:Joystick
Connections:
- net at U1.A0 (D18/ADC[7]): now also U?.~ (VCC)
- net at U1.A1 (D19/ADC[6]): now also U?.~ (VCC)
- net at U1.~ (~RESET): now also SW?.1
Changed lines of the file:
@@
 Wire Wire Line
 	11500 11350 11500 10800
+$Comp
+L Device:Joystick U?
+U 1 1 5EE6A12F
+P 2800 9300
+F 0 "U?" H 3428 9404 50  0000 L CNN
+F 1 "Joystick" H 3428 9313 50  0000 L CNN
+F 2 "" H 2650 9300 50  0001 C CNN
+F 3 "" H 2650 9300 50  0001 C CNN
+	1    2800 9300
+	1    0    0    -1
+$EndComp
+Wire Wire Line
+	2650 6900 2650 8600
+Wire Wire Line
+	2850 8600 2850 7100
+Wire Wire Line
+	2850 7100 2750 7100
+Wire Wire Line
+	2750 7100 2750 6900
 $EndSCHEMATC

Commit message: chenges
Parts:
- removed U?: Joystick, symbol Device:Joystick
- added U?: Adafruit_Ultimate_GPS, symbol Device:Adafruit_Ultimate_GPS
- added U?: dp_joystick, symbol Device:dp_joystick
Connections:
- net at U1.A2 (D20/ADC[5]): now also U?.~ (WY)
- net at U1.A3 (D21/ADC[4]): now also U?.~ (WY)
- net at U1.~ (~RESET): now also U?.~ (WY)
- net at RV?.1, SW?.1 (A), SW?.2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: now also U?.~ (WY)
- new net: U0.~ (VIN), U?.~ (VIN) (x2)
Changed lines of the file:
@@
 	3450 6900 3450 7150
 Wire Wire Line
-	3450 7150 5200 7150
+	3450 7150 3550 7150
 Wire Wire Line
 	5200 7150 5200 4300
@@
 	11500 11350 11500 10800
 $Comp
-L Device:Joystick U?
-U 1 1 5EE6A12F
-P 2800 9300
-F 0 "U?" H 3428 9404 50  0000 L CNN
-F 1 "Joystick" H 3428 9313 50  0000 L CNN
-F 2 "" H 2650 9300 50  0001 C CNN
-F 3 "" H 2650 9300 50  0001 C CNN
-	1    2800 9300
-	1    0    0    -1
-$EndComp
-Wire Wire Line
-	2650 6900 2650 8600
-Wire Wire Line
-	2850 8600 2850 7100
-Wire Wire Line
-	2850 7100 2750 7100
-Wire Wire Line
-	2750 7100 2750 6900
+L Device:Adafruit_Ultimate_GPS U?
+U 1 1 5EE87A51
+P 3400 11350
+F 0 "U?" V 2775 10658 50  0000 C CNN
+F 1 "Adafruit_Ultimate_GPS" V 2866 10658 50  0000 C CNN
+F 2 "" H 2950 9700 50  0001 C CNN
+F 3 "" H 2950 9700 50  0001 C CNN
+	1    3400 11350
+	0    1    1    0
+$EndComp
+Wire Wire Line
+	9550 6050 7950 6050
+Wire Wire Line
+	7950 6050 7950 11650
+Wire Wire Line
+	7950 11650 3500 11650
+Wire Wire Line
+	9350 8650 8050 8650
+Wire Wire Line
+	8050 8650 8050 11550
+Wire Wire Line
+	8050 11550 3500 11550
+$Comp
+L Device:dp_joystick U?
+U 1 1 5EF4B780
+P 2850 8650
+F 0 "U?" H 2322 8754 50  0000 R CNN
+F 1 "dp_joystick" H 2322 8663 50  0000 R CNN
+F 2 "" H 4350 9700 50  0001 C CNN
+F 3 "" H 4350 9700 50  0001 C CNN
+	1    2850 8650
+	1    0    0    -1
+$EndComp
+Wire Wire Line
+	2850 8050 2850 6900
+Wire Wire Line
+	3450 8650 3600 8650
+Wire Wire Line
+	3600 8650 3600 7700
+Wire Wire Line
+	3600 7700 2950 7700
+Wire Wire Line
+	2950 7700 2950 6900
+Wire Wire Line
+	2700 8050 2700 7850
+Wire Wire Line
+	2700 7850 3500 7850
+Wire Wire Line
+	3650 7850 3650 6900
+Wire Wire Line
+	3450 8500 3500 8500
+Wire Wire Line
+	3500 8500 3500 7850
+Connection ~ 3500 7850
+Wire Wire Line
+	3500 7850 3650 7850
+Wire Wire Line
+	3000 8050 3000 7550
+Wire Wire Line
+	3000 7550 3550 7550
+Wire Wire Line
+	3550 7550 3550 7150
+Connection ~ 3550 7150
+Wire Wire Line
+	3550 7150 5200 7150
+Wire Wire Line
+	3450 8800 3550 8800
+Wire Wire Line
+	3550 8800 3550 7550
+Connection ~ 3550 7550
 $EndSCHEMATC
